Commit message: added nav2 integration

File: vacbot/urdf/ros2_control.xacro (robot description, xacro)
@@ -1,3 +1,36 @@
 <?xml version="1.0"?>
 <robot xmlns:xacro="http://ros.org/wiki/xacro">
+    <ros2_control name="realSystem" type="system">
+        <!-- <hardware>
+            <plugin>mock_components/GenericSystem</plugin>
+        </hardware> -->
+        <hardware>
+            <plugin>gz_ros2_control/GazeboSimSystem</plugin>
+        </hardware>
+        <!-- <hardware>
+            <plugin>vacbot_hardware_interface/VacbotInterface</plugin>
+            <param name="left_wheel_name">left_wheel_joint</param>
+            <param name="left_forward_pin">22</param>
+            <param name="left_backward_pin">21</param>
+            <param name="left_pwm_pin">26</param>
+            <param name="right_wheel_name">right_wheel_joint</param>
+            <param name="right_forward_pin">25</param>
+            <param name="right_backward_pin">24</param>
+            <param name="right_pwm_pin">23</param>
+        </hardware> -->
+        <joint name="left_wheel_joint">
+            <command_interface name="velocity"/>
+                <param name="min">-1</param>
+                <param name="max">1</param>
+            <state_interface name="position"/>
+            <state_interface name="velocity"/>
+        </joint>
+        <joint name="right_wheel_joint">
+            <command_interface name="velocity"/>
+                <param name="min">-1</param>
+                <param name="max">1</param>
+            <state_interface name="position"/>
+            <state_interface name="velocity"/>
+        </joint>
+    </ros2_control>
 </robot>

File: vacbot/urdf/vacbot.urdf.xacro (robot description, xacro)
@@ -1,6 +1,6 @@
 <?xml version="1.0"?>
 <robot name="vac_bot" xmlns:xacro="http://ros.org/wiki/xacro">
-    <xacro:property name="base_radius" value="0.150"/>
-    <xacro:property name="base_height" value="0.068"/>
+    <xacro:property name="chassis_radius" value="0.150"/>
+    <xacro:property name="chassis_height" value="0.068"/>
     <xacro:property name="wheel_radius" value="0.0215"/>
     <xacro:property name="wheel_width" value="0.018"/>
@@ -11,72 +11,175 @@
     <xacro:property name="caster_dz" value="-0.0350625"/>
     <xacro:property name="caster_radius" value="0.0079375"/>
-    <link name="base_link">
-        <visual>
-        <geometry>
-            <cylinder radius="${base_radius}" length="${base_height}"/>
-        </geometry>
-        <material name="Cyan">
-            <color rgba="0 1.0 1.0 0.5"/>
-        </material>
-        </visual>
-    </link>
+    <xacro:macro name="box_inertia" params="m w h d">
+        <inertial>
+            <origin xyz="0 0 0" rpy="${pi/2} 0 ${pi/2}"/>
+            <mass value="${m}"/>
+            <inertia ixx="${(m/12) * (h*h + d*d)}" ixy="0.0" ixz="0.0" iyy="${(m/12) * (w*w + d*d)}" iyz="0.0" izz="${(m/12) * (w*w + h*h)}"/>
+        </inertial>
+    </xacro:macro>
+    <xacro:macro name="cylinder_inertia" params="m r h">
+        <inertial>
+            <origin xyz="0 0 0" rpy="${pi/2} 0 0" />
+            <mass value="${m}"/>
+            <inertia ixx="${(m/12) * (3*r*r + h*h)}" ixy = "0" ixz = "0" iyy="${(m/12) * (3*r*r + h*h)}" iyz = "0" izz="${(m/2) * (r*r)}"/>
+        </inertial>
+    </xacro:macro>
+    <xacro:macro name="sphere_inertia" params="m r">
+        <inertial>
+            <mass value="${m}"/>
+            <inertia ixx="${(2/5) * m * (r*r)}" ixy="0.0" ixz="0.0" iyy="${(2/5) * m * (r*r)}" iyz="0.0" izz="${(2/5) * m * (r*r)}"/>
+        </inertial>
+    </xacro:macro>
+    <link name="base_link"/>
     <link name="base_footprint"/>
-    <joint name="base_joint" type="fixed">
+    <joint name="base_footprint_joint" type="fixed">
         <parent link="base_link"/>
         <child link="base_footprint"/>
-        <origin xyz="0.0 0.0 ${0.11}" rpy="0 0 0"/>
+        <origin xyz="0 0 0" rpy="0 0 0"/>
+    </joint>
+    <link name="chassis">
+        <visual>
+            <geometry>
+                <cylinder radius="${chassis_radius}" length="${chassis_height}"/>
+            </geometry>
+            <material name="Cyan">
+                <color rgba="0 1.0 1.0 0.5"/>
+            </material>
+        </visual>
+        <collision>
+            <origin xyz="0 0 0" rpy="${pi/2} 0 0"/>
+            <geometry>
+                <box size="${chassis_radius*2.0} ${chassis_height} ${chassis_radius*2.0}"/>
+                <cylinder radius="${chassis_radius}" length="${chassis_height}"/>
+            </geometry>
+        </collision>
+        <xacro:box_inertia m="1" w="${chassis_radius*2}" d="${chassis_radius*2}" h="${chassis_height}"/>
+    </link>
+    <joint name="chassis_joint" type="fixed">
+        <parent link="base_link"/>
+        <child link="chassis"/>
+        <origin xyz="0 0 0"/>
     </joint>
     <link name="left_wheel_link">
         <visual>
-        <origin xyz="0 0 0" rpy="${pi/2} 0 0"/>
-        <geometry>
-            <cylinder radius="${wheel_radius}" length="${wheel_width}"/>
-        </geometry>
-        <material name="Gray">
-            <color rgba="0.5 0.5 0.5 1.0"/>
-        </material>
-        </visual>
+            <origin xyz="0 0 0" rpy="0 0 0"/>
+            <geometry>
+                <cylinder radius="${wheel_radius}" length="${wheel_width}"/>
+            </geometry>
+            <material name="Gray">
+                <color rgba="0.5 0.5 0.5 1.0"/>
+            </material>
+        </visual>
+        <collision>
+            <origin xyz="0 0 0" rpy="0 0 0"/>
+            <geometry>
+                <cylinder radius="${wheel_radius}" length="${wheel_width}"/>
+            </geometry>
+        </collision>
+        <xacro:cylinder_inertia m="0.01" r="${wheel_radius}" h="${wheel_width}"/>
     </link>
     <link name="right_wheel_link">
-        <visual>
-        <origin xyz="0 0 0" rpy="${pi/2} 0 0"/>
-        <geometry>
-            <cylinder radius="${wheel_radius}" length="${wheel_width}"/>
-        </geometry>
-        <material name="Gray">
-            <color rgba="0.5 0.5 0.5 1.0"/>
-        </material>
-        </visual>
+            <visual>
+            <origin xyz="0 0 0" rpy="0 0 0"/>
+            <geometry>
+                <cylinder radius="${wheel_radius}" length="${wheel_width}"/>
+            </geometry>
+            <material name="Gray">
+                <color rgba="0.5 0.5 0.5 1.0"/>
+            </material>
+        </visual>
+        <collision>
+            <origin xyz="0 0 0" rpy="0 0 0"/>
+            <geometry>
+                <cylinder radius="${wheel_radius}" length="${wheel_width}"/>
+            </geometry>
+        </collision>
+        <xacro:cylinder_inertia m="0.01" r="${wheel_radius}" h="${wheel_width}"/>
     </link>
     <joint name="left_wheel_joint" type="continuous">
-        <parent link="base_link"/>
+        <parent link="chassis"/>
         <child link="left_wheel_link"/>
-        <origin xyz="${wheel_dx} ${wheel_dy} ${wheel_dz}" rpy="0 0 0"/>
+        <origin xyz="${wheel_dx} ${wheel_dy} ${wheel_dz}" rpy="-${pi/2} 0 0"/>
+        <axis xyz="0 0 1"/>
     </joint>
     <joint name="right_wheel_joint" type="continuous">
-        <parent link="base_link"/>
+        <parent link="chassis"/>
         <child link="right_wheel_link"/>
-        <origin xyz="${wheel_dx} ${-wheel_dy} ${wheel_dz}" rpy="0 0 0"/>
+        <origin xyz="${wheel_dx} ${-wheel_dy} ${wheel_dz}" rpy="-${pi/2} 0 0"/>
+        <axis xyz="0 0 1"/>
     </joint>
     <link name="front_caster">
         <visual>
-        <geometry>
-            <sphere radius="${caster_radius}"/>
-        </geometry>
-        <material name="Cyan">
-            <color rgba="0 1.0 1.0 1.0"/>
-        </material>
-        </visual>
+            <geometry>
+                <sphere radius="${caster_radius}"/>
+            </geometry>
+            <material name="Cyan">
+                <color rgba="0 1.0 1.0 1.0"/>
+            </material>
+        </visual>
+        <collision>
+            <origin xyz="0 0 0" rpy="0 0 0"/>
+            <geometry>
+                <sphere radius="${caster_radius}"/>
+            </geometry>
+        </collision>
+        <xacro:sphere_inertia m="0.005" r="${caster_radius}"/>
     </link>
     <joint name="caster_joint" type="fixed">
-        <parent link="base_link"/>
+        <parent link="chassis"/>
         <child link="front_caster"/>
         <origin xyz="${caster_dx} 0.0 ${caster_dz}" rpy="0 0 0"/>
     </joint>
-    <ros2_control name="realSystem" type="system">
+    <link name="lidar_link">
+        <inertial>
+            <origin xyz="0 0 0" rpy="0 0 0"/>
+            <mass value="0.125"/>
+            <inertia ixx="0.001"  ixy="0"  ixz="0" iyy="0.001" iyz="0" izz="0.001" />
+        </inertial>
+        <collision>
+            <origin xyz="0 0 0" rpy="0 0 0"/>
+            <geometry>
+                <cylinder radius="0.035" length="0.025"/>
+            </geometry>
+        </collision>
+        <visual>
+            <origin xyz="0 0 0" rpy="0 0 0"/>
+            <geometry>
+                <cylinder radius="0.035" length="0.025"/>
+            </geometry>
+        </visual>
+    </link>
+    <joint name="lidar_joint" type="fixed">
+        <parent link="base_link"/>
+        <child link="lidar_link"/>
+        <origin xyz="0.06 0 0.0465" rpy="0 -0.04 0"/>
+    </joint>
+    <gazebo reference="lidar_link">
+        <sensor name="laser" type="gpu_lidar">
+            <pose> 0 0 0 0 0 0 </pose>
+            <visualize>true</visualize>
+            <update_rate>10</update_rate>
+            <lidar>
+                <scan>
+                    <horizontal>
+                        <samples>360</samples>
+                        <min_angle>-3.14</min_angle>
+                        <max_angle>3.14</max_angle>
+                    </horizontal>
+                </scan>
+                <range>
+                    <min>0.15</min>
+                    <max>12</max>
+                </range>
+            </lidar>
+            <topic>scan</topic>
+            <gz_frame_id>lidar_link</gz_frame_id>
+        </sensor>
+    </gazebo>
+    <ros2_control name="GazeboSimSystem" type="system">
+        <hardware>
+            <plugin>gz_ros2_control/GazeboSimSystem</plugin>
+        </hardware>
         <!-- <hardware>
-            <plugin>mock_components/GenericSystem</plugin>
-        </hardware> -->
-        <hardware>
             <plugin>vacbot_hardware_interface/VacbotInterface</plugin>
             <param name="left_wheel_name">left_wheel_joint</param>
@@ -88,13 +191,26 @@
             <param name="right_backward_pin">24</param>
             <param name="right_pwm_pin">23</param>
-        </hardware>
+        </hardware> -->
         <joint name="left_wheel_joint">
             <command_interface name="velocity"/>
             <state_interface name="position"/>
+            <state_interface name="velocity"/>
         </joint>
         <joint name="right_wheel_joint">
             <command_interface name="velocity"/>
             <state_interface name="position"/>
+            <state_interface name="velocity"/>
         </joint>
     </ros2_control>
+    <gazebo>
+        <plugin filename="gz_ros2_control-system" name="gz_ros2_control::GazeboSimROS2ControlPlugin">
+            <parameters>$(find vacbot)/config/ros2_controllers.yaml</parameters>
+        </plugin>
+        <plugin filename="gz-sim-joint-state-publisher-system"
+            name="gz::sim::systems::JointStatePublisher">
+            <topic>joint_states</topic>
+            <joint_name>left_wheel_joint</joint_name>
+            <joint_name>right_wheel_joint</joint_name>
+        </plugin>
+    </gazebo>
 </robot>

File: vacbot/urdf/vacbot_description.urdf (robot description, URDF)
Before this commit: robot None, 5 links, 4 joints
Links:
- link base_link: geometry collision box size=${base_radius*2.0} ${base_height} ${base_radius*2.0}; visual cylinder length=${base_height} radius=${base_radius}
- link front_caster: geometry collision sphere radius=${caster_radius}; visual sphere radius=${caster_radius}
- link left_wheel_link: geometry collision cylinder length=${wheel_width} radius=${wheel_radius}; visual cylinder length=${wheel_width} radius=${wheel_radius}
- link right_wheel_link: geometry collision cylinder length=${wheel_width} radius=${wheel_radius}; visual cylinder length=${wheel_width} radius=${wheel_radius}
